Commit message: add multiple obstacles

File: push-policy/push_policy/resources/obstacle2.urdf (robot description, URDF)
Before this commit: robot obstacle1, 1 links, 0 joints
Links:
- link base_link: mass 0.6 -> 0.5; geometry collision box size=0.45 0.25 0.25; visual box size=0.45 0.25 0.25

File: push-policy/push_policy/resources/obstacle3.urdf (robot description, URDF)
Before this commit: robot obstacle1, 1 links, 0 joints
Links:
- link base_link: mass 0.6 -> 0.7; geometry collision cylinder length=0.25 radius=0.4; visual cylinder length=0.25 radius=0.4

File: push-policy/push_policy/resources/obstacle4.urdf (robot description, URDF)
Before this commit: robot obstacle1, 1 links, 0 joints
Links:
- link base_link: mass 0.6 -> 0.4; geometry collision box size=0.45 0.35 0.25; visual box size=0.45 0.35 0.25

File: push-policy/push_policy/resources/obstacle5.urdf (robot description, URDF)
Before this commit: robot obstacle1, 1 links, 0 joints
Links:
- link base_link: mass 0.6 -> 0.1; geometry collision cylinder length=0.4 radius=0.4; visual cylinder length=0.4 radius=0.4
