Commit message: add moment of inertia

File: push-policy/push_policy/resources/obstacle1.urdf (robot description, URDF)
Before this commit: robot obstacle1, 1 links, 0 joints
Links:
- link base_link: mass 0.6 -> 2; geometry collision cylinder length=0.25 radius=0.4; visual cylinder length=0.25 radius=0.4

File: push-policy/push_policy/resources/obstacle2.urdf (robot description, URDF)
Before this commit: robot obstacle2, 1 links, 0 joints
Links:
- link base_link: mass 0.5 -> 3

File: push-policy/push_policy/resources/obstacle3.urdf (robot description, URDF)
Before this commit: robot obstacle3, 1 links, 0 joints
Links:
- link base_link: mass 0.7 -> 4

File: push-policy/push_policy/resources/obstacle4.urdf (robot description, URDF)
Before this commit: robot obstacle2, 1 links, 0 joints
Links:
- link base_link: mass 0.4 -> 100

File: push-policy/push_policy/resources/obstacle5.urdf (robot description, URDF)
Before this commit: robot obstacle3, 1 links, 0 joints
Links:
- link base_link: mass 0.1 -> 4.5
